File: Hardware/kicad/C4-Clock.kicad_sch (KiCad schematic)
At the start: 24 parts, among them J1 Keypad, J2 Battery, J3 LCD1602, J4 Boost Module, K1 FINDER-36.11-5V, Q1 S9014, Q2 S9014, SW1 SW_SPST, SW2 SW_SPST, U1 ATmega328P-P, U2 AMS1117-5.0, U3 PCF8574A, Y1 16MHz

Commit message: kicad: create PCB
Parts:
- added BT1: CR2032, Battery:BatteryHolder_ComfortableElectronic_CH273-2450_1x2450, symbol Device:Battery_Cell
- added J5: ICSP, Connector_PinHeader_2.54mm:PinHeader_2x03_P2.54mm_Vertical, symbol Connector_Generic:Conn_02x03_Odd_Even
- added U4: DS1302+, Package_DIP:DIP-8_W7.62mm, symbol Timer_RTC:DS1302+
- added Y2: 32.768kHz, Crystal:Crystal_AT310_D3.0mm_L10.0mm_Horizontal, symbol Device:Crystal
- BZ1: footprint (none) -> Buzzer_Beeper:Buzzer_12x9.5RM7.6
- C1, C2: footprint Capacitor_THT:C_Disc_D3.0mm_W1.6mm_P2.50mm -> Capacitor_THT:C_Disc_D4.3mm_W1.9mm_P5.00mm
- C4: footprint (none) -> Capacitor_THT:C_Disc_D4.3mm_W1.9mm_P5.00mm
- D1: footprint (none) -> LED_THT:LED_D5.0mm
- D2: footprint (none) -> Diode_THT:D_A-405_P7.62mm_Horizontal
- J4: footprint (none) -> DC-Buck:DC-Buck-2A
- R3: footprint Resistor_THT:R_Axial_DIN0207_L6.3mm_D2.5mm_P10.16mm_Horizontal -> Potentiometer_THT:Potentiometer_Vishay_T73YP_Vertical
- SW2: footprint Button_Switch_THT:SW_E-Switch_EG1271_DPDT -> Button_Switch_THT:SW_Push_2P2T_Toggle_CK_PVA2xxH1xxxxxxV2
- U1: footprint Package_DIP:DIP-28_W7.62mm -> Package_DIP:DIP-28_W7.62mm_Socket
- Y1: footprint (none) -> Crystal:Crystal_HC49-4H_Vertical
Connections:
- net +5V: now also J5.2 (Pin_2), U4.8 (VCC1)
- net GND: now also C3.1, BT1.2 (-), J5.6 (Pin_6), U4.4 (GND); no longer C3.2
- net LED: now also U1.23 (PC0); no longer U1.17 (PB3)
- net RELAY: now also U1.24 (PC1); no longer U1.18 (PB4)
- net at U2.3 (VI): now also SW1.2 (B)
- net RESET: now reaches U1.1 (~{RESET}/PC6)
- net RESET: now also J5.5 (Pin_5)
- net PB5: now reaches U1.19 (PB5)
- net PB5: now also J5.3 (Pin_3), U4.5 (CE)
- net at K1.11: now also C3.2; no longer C3.1
- new net: BT1.1 (+), U4.1 (VCC2)
- new net: U4.2 (X1), Y2.2
- new net: U4.3 (X2), Y2.1
- new net PB3: J5.4 (Pin_4), U1.17 (PB3), U4.7 (SCLK)
- new net PB4: J5.1 (Pin_1), U1.18 (PB4), U4.6 (I/O)
Other:
- note added: "<- May use this to deactivate the "bomb" physically"
- note removed: "<- May use this to deactivate the "bomb"."
- moved on the sheet: C3, C4, D1, R4

Commit message: doc: Add lcd1602 reference
Parts:
- removed D2: 1N4001, Diode_THT:D_A-405_P7.62mm_Horizontal, symbol Device:D
- added D2, D3: 1N4001, Diode_THT:D_DO-41_SOD81_P10.16mm_Horizontal, symbol Diode:1N4001
- added H1, H3, H5, H7: LCD1602, MountingHole:MountingHole_3mm_Pad_TopBottom, symbol Mechanical:MountingHole_Pad
- added H2, H4, H6, H8: hole, MountingHole:MountingHole_3mm_Pad_TopBottom, symbol Mechanical:MountingHole_Pad
Connections:
- net +8V: now also D2.2 (A); no longer J2.1 (Pin_1)
- net GND: now also D3.2 (A), H1.1, H2.1, H3.1, H4.1, H5.1, H6.1, H7.1, H8.1
- net RELAY: now also D3.1 (K)
- new net: D2.1 (K), J2.1 (Pin_1)

Commit message: software: Added VS files
Parts:
- added Q3: S9014, Package_TO_SOT_THT:TO-92, symbol Device:Q_NPN_EBC
- added R5: 1k, Resistor_THT:R_Axial_DIN0207_L6.3mm_D2.5mm_P10.16mm_Horizontal, symbol Device:R
Connections:
- net +5V: now also Q3.3 (C)
- net RELAY: now also R5.1; no longer D3.1 (K), K1.A1
- new net: Q3.2 (B), R5.2
- new net: D3.1 (K), K1.A1, Q3.1 (E)
Changed lines of the file:
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@@
     )
   )
-  (global_label "RELAY" (shape input) (at 228.6 62.23 180) (fields_autoplaced)
+  (global_label "RELAY" (shape input) (at 213.36 57.15 180) (fields_autoplaced)
     (effects (font (size 1.27 1.27)) (justify right))
-    (property "Intersheet References" "${INTERSHEET_REFS}" (id 0) (at 220.6515 62.1506 0)
+    (property "Intersheet References" "${INTERSHEET_REFS}" (id 0) (at 205.4115 57.0706 0)
       (effects (font (size 1.27 1.27)) (justify right) hide)
     )
@@
     )
     (pin "1")
+  )
+  (symbol (lib_id "Device:R") (at 217.17 57.15 90) (unit 1)
+    (in_bom yes) (on_board yes) (fields_autoplaced)
+    (property "Reference" "R5" (id 0) (at 217.17 50.8 90))
+    (property "Value" "1k" (id 1) (at 217.17 53.34 90))
+    (property "Footprint" "Resistor_THT:R_Axial_DIN0207_L6.3mm_D2.5mm_P10.16mm_Horizontal" (id 2) (at 217.17 58.928 90)
+      (effects (font (size 1.27 1.27)) hide)
+    )
+    (property "Datasheet" "~" (id 3) (at 217.17 57.15 0)
+      (effects (font (size 1.27 1.27)) hide)
+    )
+    (pin "1")
+    (pin "2")
   )
   (symbol (lib_id "power:+8V") (at 105.41 20.32 0) (unit 1)
@@
     (pin "1")
   )
+  (symbol (lib_id "Device:Q_NPN_EBC") (at 226.06 57.15 0) (unit 1)
+    (in_bom yes) (on_board yes) (fields_autoplaced)
+    (property "Reference" "Q3" (id 0) (at 231.14 55.8799 0)
+      (effects (font (size 1.27 1.27)) (justify left))
+    )
+    (property "Value" "S9014" (id 1) (at 231.14 58.4199 0)
+      (effects (font (size 1.27 1.27)) (justify left))
+    )
+    (property "Footprint" "Package_TO_SOT_THT:TO-92" (id 2) (at 231.14 54.61 0)
+      (effects (font (size 1.27 1.27)) hide)
+    )
+    (property "Datasheet" "~" (id 3) (at 226.06 57.15 0)
+      (effects (font (size 1.27 1.27)) hide)
+    )
+    (pin "1")
+    (pin "2")
+    (pin "3")
+  )
   (symbol (lib_id "Relay:FINDER-36.11") (at 233.68 76.2 0) (unit 1)
     (in_bom yes) (on_board yes) (fields_autoplaced)
@@
     (pin "2")
   )
+  (symbol (lib_id "power:+5V") (at 228.6 52.07 0) (unit 1)
+    (in_bom yes) (on_board yes) (fields_autoplaced)
+    (property "Reference" "#PWR036" (id 0) (at 228.6 55.88 0)
+      (effects (font (size 1.27 1.27)) hide)
+    )
+    (property "Value" "+5V" (id 1) (at 228.6 46.99 0))
+    (property "Footprint" "" (id 2) (at 228.6 52.07 0)
+      (effects (font (size 1.27 1.27)) hide)
+    )
+    (property "Datasheet" "" (id 3) (at 228.6 52.07 0)
+      (effects (font (size 1.27 1.27)) hide)
+    )
+    (pin "1")
+  )
   (symbol (lib_id "Mechanical:MountingHole_Pad") (at 236.22 111.76 0) (unit 1)
     (in_bom yes) (on_board yes) (fields_autoplaced)
@@
       (reference "#PWR035") (unit 1) (value "GND") (footprint "")
     )
+    (path "/ad71b609-e7e1-4666-9fd0-6d88c7d96f36"
+      (reference "#PWR036") (unit 1) (value "+5V") (footprint "")
+    )
     (path "/4175d047-bf8f-4806-a5bb-cf208b2718be"
       (reference "BT1") (unit 1) (value "CR2032") (footprint "Battery:BatteryHolder_ComfortableElectronic_CH273-2450_1x2450")
@@
       (reference "Q2") (unit 1) (value "S9014") (footprint "Package_TO_SOT_THT:TO-92")
     )
+    (path "/4c6510d9-017e-4c47-82ba-5105026c6f89"
+      (reference "Q3") (unit 1) (value "S9014") (footprint "Package_TO_SOT_THT:TO-92")
+    )
     (path "/a9d015c2-a71b-46ad-b3a4-6eea7301ee51"
       (reference "R1") (unit 1) (value "1k") (footprint "Resistor_THT:R_Axial_DIN0207_L6.3mm_D2.5mm_P10.16mm_Horizontal")
@@
       (reference "R4") (unit 1) (value "220") (footprint "Resistor_THT:R_Axial_DIN0207_L6.3mm_D2.5mm_P10.16mm_Horizontal")
     )
+    (path "/206bfdd0-417d-49a5-beaa-7015cee73d7c"
+      (reference "R5") (unit 1) (value "1k") (footprint "Resistor_THT:R_Axial_DIN0207_L6.3mm_D2.5mm_P10.16mm_Horizontal")
+    )
     (path "/48e61d41-43dc-4080-9b7f-b92302b5ae95"

Commit message: hardware: Update PCB
Parts:
- U4: footprint Package_DIP:DIP-8_W7.62mm -> Package_DIP:DIP-8_W7.62mm_Socket
Connections:
- net +8V: now also D2.1 (K); no longer D2.2 (A)
- net PB3: now also U4.5 (CE); no longer U4.7 (SCLK)
- net PB4: no longer U4.6 (I/O)
- net PB5: no longer U4.5 (CE)
- net at J2.1 (Pin_1): now also D2.2 (A); no longer D2.1 (K)
- net DS1302_CLK: now reaches U1.25 (PC2)
- net DS1302_CLK: now also U4.7 (SCLK)
- net DS1302_IO: now reaches U1.26 (PC3)
- net DS1302_IO: now also U4.6 (I/O)
Other:
- moved on the sheet: D2
Changed lines of the file:
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@@
     )
   )
-  (global_label "PB4" (shape input) (at 85.09 151.13 0) (fields_autoplaced)
+  (global_label "DS1302_IO" (shape input) (at 85.09 151.13 0) (fields_autoplaced)
     (effects (font (size 1.27 1.27)) (justify left))
-    (property "Intersheet References" "${INTERSHEET_REFS}" (id 0) (at 91.1637 151.0506 0)
+    (property "Intersheet References" "${INTERSHEET_REFS}" (id 0) (at 97.6347 151.0506 0)
       (effects (font (size 1.27 1.27)) (justify left) hide)
     )
@@
     )
   )
+  (global_label "DS1302_IO" (shape output) (at 85.09 86.36 0) (fields_autoplaced)
+    (effects (font (size 1.27 1.27)) (justify left))
+    (property "Intersheet References" "${INTERSHEET_REFS}" (id 0) (at 97.6347 86.2806 0)
+      (effects (font (size 1.27 1.27)) (justify left) hide)
+    )
+  )
   (global_label "BUZZER" (shape input) (at 139.7 113.03 180) (fields_autoplaced)
     (effects (font (size 1.27 1.27)) (justify right))
@@
     )
   )
-  (global_label "PB5" (shape input) (at 59.69 153.67 180) (fields_autoplaced)
+  (global_label "PB3" (shape input) (at 59.69 153.67 180) (fields_autoplaced)
     (effects (font (size 1.27 1.27)) (justify right))
     (property "Intersheet References" "${INTERSHEET_REFS}" (id 0) (at 53.6163 153.5906 0)
       (effects (font (size 1.27 1.27)) (justify right) hide)
+    )
+  )
+  (global_label "DS1302_CLK" (shape output) (at 85.09 83.82 0) (fields_autoplaced)
+    (effects (font (size 1.27 1.27)) (justify left))
+    (property "Intersheet References" "${INTERSHEET_REFS}" (id 0) (at 99.2675 83.7406 0)
+      (effects (font (size 1.27 1.27)) (justify left) hide)
     )
   )
@@
     )
   )
-  (global_label "PB3" (shape input) (at 59.69 151.13 180) (fields_autoplaced)
+  (global_label "DS1302_CLK" (shape input) (at 59.69 151.13 180) (fields_autoplaced)
     (effects (font (size 1.27 1.27)) (justify right))
-    (property "Intersheet References" "${INTERSHEET_REFS}" (id 0) (at 53.6163 151.0506 0)
+    (property "Intersheet References" "${INTERSHEET_REFS}" (id 0) (at 45.5125 151.0506 0)
       (effects (font (size 1.27 1.27)) (justify right) hide)
     )
@@
     (pin "1")
   )
-  (symbol (lib_id "Diode:1N4001") (at 105.41 22.86 90) (unit 1)
+  (symbol (lib_id "Diode:1N4001") (at 105.41 22.86 270) (unit 1)
     (in_bom yes) (on_board yes) (fields_autoplaced)
     (property "Reference" "D2" (id 0) (at 107.95 21.5899 90)
-      (effects (font (size 1.27 1.27)) (justify right))
+      (effects (font (size 1.27 1.27)) (justify left))
     )
     (property "Value" "1N4001" (id 1) (at 107.95 24.1299 90)
-      (effects (font (size 1.27 1.27)) (justify right))
-    )
-    (property "Footprint" "Diode_THT:D_DO-41_SOD81_P10.16mm_Horizontal" (id 2) (at 109.855 22.86 0)
+      (effects (font (size 1.27 1.27)) (justify left))
+    )
+    (property "Footprint" "Diode_THT:D_DO-41_SOD81_P10.16mm_Horizontal" (id 2) (at 100.965 22.86 0)
       (effects (font (size 1.27 1.27)) hide)
     )
@@
     (property "Reference" "U4" (id 0) (at 82.55 144.78 0))
     (property "Value" "DS1302+" (id 1) (at 82.55 147.32 0))
-    (property "Footprint" "Package_DIP:DIP-8_W7.62mm" (id 2) (at 72.39 168.91 0)
+    (property "Footprint" "Package_DIP:DIP-8_W7.62mm_Socket" (id 2) (at 72.39 168.91 0)
       (effects (font (size 1.27 1.27)) hide)
     )
@@
     )
     (path "/9c8b409b-0d1b-49e5-8fed-acd83e0e8b3e"
-      (reference "U4") (unit 1) (value "DS1302+") (footprint "Package_DIP:DIP-8_W7.62mm")
+      (reference "U4") (unit 1) (value "DS1302+") (footprint "Package_DIP:DIP-8_W7.62mm_Socket")
     )
     (path "/00000000-0000-0000-0000-0000621ca23f"
